File: HomeAutomation.kicad_sch (KiCad schematic)
At the start: 28 parts, among them J1 Conn_01x04, J2 Screw_Terminal_01x04, J3 Screw_Terminal_01x03, K1 PR13-5V-450-1C, K2 RAYEX-L90AS, Q1 S8050, Q2 S8050, SW1 SW_Push, SW2 SW_Push, U1 ESP32-WROOM-32, U2 PC817, U3 PC817, U4 AMS1117-3.3, U5 HLK-PM01

Commit message: Completed Project
Parts:
- added H1, H2, H3, H4: MountingHole, MountingHole:MountingHole_2.7mm_M2.5_Pad_Via, symbol Mechanical:MountingHole
- C1, C2: footprint (none) -> Capacitor_SMD:C_0805_2012Metric
- D1, D2: footprint (none) -> LED_SMD:LED_0805_2012Metric
- J1: footprint (none) -> Connector_PinHeader_2.54mm:PinHeader_1x04_P2.54mm_Vertical
- J2: footprint (none) -> TerminalBlock:TerminalBlock_MaiXu_MX126-5.0-04P_1x04_P5.00mm
- J3: footprint (none) -> TerminalBlock:TerminalBlock_MaiXu_MX126-5.0-03P_1x03_P5.00mm
- K1: footprint PR13-5V-450-1C:RELAY_PR13-5V-450-1C -> PR13-5V-450-1C_footprint:RELAY_PR13-5V-450-1C
- R1, R2, R3, R4, R5, R6, R7, R8: footprint (none) -> Resistor_SMD:R_0805_2012Metric
- SW1, SW2: footprint (none) -> Button_Switch_THT:SW_PUSH_6mm
